File: connectors.kicad_sch (KiCad schematic)
At the start: 34 parts, among them J10 Conn_01x02, J11 Conn_01x02, J12 Conn_01x02, J13 USB_C_Receptacle_PowerOnly_6P, J14 USB_C_Receptacle_USB2.0_16P, J15 USB_C_Receptacle_USB2.0_16P, J3 VIN, J4 Conn_01x08, J5 Conn_01x08, J6 Conn_01x08, J7 Conn_01x02, J8 Conn_01x02, J9 Conn_01x02

Commit message: silinecek
Parts:
- removed J4, J5, J6: Conn_01x08, Connector_PinHeader_2.54mm:PinHeader_1x08_P2.54mm_Vertical, symbol Connector_Generic:Conn_01x08
- removed R38, R39, R40: 12k, Resistor_SMD:R_0805_2012Metric, symbol Device:R_Small
- added C42: 220uF 35V, Capacitor_SMD:CP_Elec_8x10.5, symbol Device:C_Polarized_Small
- added J14: Servo2, Connector_JST:JST_XA_B03B-XASK-1_1x03_P2.50mm_Vertical, symbol Connector_Generic:Conn_01x03
- added J15: Servo4, Connector_JST:JST_XA_B03B-XASK-1_1x03_P2.50mm_Vertical, symbol Connector_Generic:Conn_01x03
- added J16: Servo6, Connector_JST:JST_XA_B03B-XASK-1_1x03_P2.50mm_Vertical, symbol Connector_Generic:Conn_01x03
- added J17: Servo8, Connector_JST:JST_XA_B03B-XASK-1_1x03_P2.50mm_Vertical, symbol Connector_Generic:Conn_01x03
- added J3: Servo1, Connector_JST:JST_XA_B03B-XASK-1_1x03_P2.50mm_Vertical, symbol Connector_Generic:Conn_01x03
- added J4: Servo3, Connector_JST:JST_XA_B03B-XASK-1_1x03_P2.50mm_Vertical, symbol Connector_Generic:Conn_01x03
- added J5: Servo5, Connector_JST:JST_XA_B03B-XASK-1_1x03_P2.50mm_Vertical, symbol Connector_Generic:Conn_01x03
- added J6: Servo7, Connector_JST:JST_XA_B03B-XASK-1_1x03_P2.50mm_Vertical, symbol Connector_Generic:Conn_01x03
- added R45, R46, R47: 12k, Resistor_SMD:R_0805_2012Metric, symbol Device:R_Small
- J10: renamed from J9; footprint Connector_JST:JST_XH_S2B-XH-A-1_1x02_P2.50mm_Horizontal -> Connector_JST:JST_XH_B2B-XH-A_1x02_P2.50mm_Vertical
- J11: renamed from J10; footprint Connector_JST:JST_XH_S2B-XH-A-1_1x02_P2.50mm_Horizontal -> Connector_JST:JST_XH_B2B-XH-A_1x02_P2.50mm_Vertical
- J12: renamed from J11; footprint Connector_JST:JST_XH_S2B-XH-A-1_1x02_P2.50mm_Horizontal -> Connector_JST:JST_XH_B2B-XH-A_1x02_P2.50mm_Vertical
- J13: renamed from J12; footprint Connector_JST:JST_XH_S2B-XH-A-1_1x02_P2.50mm_Horizontal -> Connector_JST:JST_XH_B2B-XH-A_1x02_P2.50mm_Vertical
- J8: renamed from J7; footprint Connector_JST:JST_XH_S2B-XH-A-1_1x02_P2.50mm_Horizontal -> Connector_JST:JST_XH_B2B-XH-A_1x02_P2.50mm_Vertical
- J9: renamed from J8; footprint Connector_JST:JST_XH_S2B-XH-A-1_1x02_P2.50mm_Horizontal -> Connector_JST:JST_XH_B2B-XH-A_1x02_P2.50mm_Vertical
- renumbered C7 to C41, D31 to D26, D26 to D27, D30 to D28, D27 to D30, D28 to D31, J13 to J18, J15 to J19, J14 to J20, J3 to J7, R37 to R40, R46 to R48, R45 to R49, R48 to R50, R47 to R51, R50 to R52, R49 to R53
Connections:
- net 5V2: now also C42.1, J14.2 (Pin_2), J15.2 (Pin_2), J16.2 (Pin_2), J17.2 (Pin_2), J3.2 (Pin_2), J4.2 (Pin_2), J5.2 (Pin_2), J6.2 (Pin_2)
- net GND: now also C42.2, J14.1 (Pin_1), J15.1 (Pin_1), J16.1 (Pin_1), J17.1 (Pin_1), J3.1 (Pin_1), J4.1 (Pin_1), J5.1 (Pin_1), J6.1 (Pin_1)
- net PCA_1: now also R44.2
- net PCA_2: now also R41.2
- net PCA_3: now also R45.2
- net PCA_4: now also R42.2; no longer R41.2
- net PCA_5: now also R46.2; no longer R42.2
- net PCA_7: now also R47.2; no longer R44.2
- net at R43.1: now also J6.3 (Pin_3)
- net at R40.1: now also J3.3 (Pin_3)
- net at R41.1: now also J4.3 (Pin_3)
- net at R42.1: now also J5.3 (Pin_3)
- net at R44.1: now also J14.3 (Pin_3)
- new net: J16.3 (Pin_3), R46.1
- new net: J17.3 (Pin_3), R47.1
- new net: J15.3 (Pin_3), R45.1
Other:
- moved on the sheet: C41, R40
