File: dc_driver.kicad_sch (KiCad schematic)
At the start: 36 parts, among them U2 L298N, U3 L298N, U4 L298N

Commit message: silinecek
Parts:
- renumbered C12 to C10, C13 to C11, C11 to C9, D36 to D13, D37 to D14, D38 to D15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
