File: gpio_exp.kicad_sch (KiCad schematic)
At the start: 23 parts, among them U11 MCP23S17_SO

Commit message: silinecek
Parts:
- renumbered R68 to R65, R69 to R66, R70 to R67, R71 to R68, R72 to R69, R73 to R70, R74 to R71, R75 to R72, R76 to R73, R77 to R74, R78 to R75, R79 to R76, R84 to R77, R80 to R78, R81 to R79, R82 to R80, R83 to R81
Changed lines of the file:
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@@
 		(on_board yes)
 		(dnp no)
-		(property "Reference" "R79"
+		(property "Reference" "R76"
 			(at 69.85 52.578 90)
 			(effects
@@
 			(project "controllerForVehicle"
 				(path "/f177fb06-71dc-4865-9331-a828b12c2bf7/cf99d41f-154f-4525-9df8-a364b4903864"
-					(reference "R79")
+					(reference "R76")
 					(unit 1)
 				)
@@
 		(on_board yes)
 		(dnp no)
-		(property "Reference" "R75"
+		(property "Reference" "R72"
 			(at 69.85 44.958 90)
 			(effects
@@
 			(project "controllerForVehicle"
 				(path "/f177fb06-71dc-4865-9331-a828b12c2bf7/cf99d41f-154f-4525-9df8-a364b4903864"
-					(reference "R75")
+					(reference "R72")
 					(unit 1)
 				)
@@
 		(dnp no)
 		(fields_autoplaced yes)
-		(property "Reference" "#PWR051"
+		(property "Reference" "#PWR057"
 			(at 50.8 90.17 0)
 			(effects
@@
 			(project "controllerForVehicle"
 				(path "/f177fb06-71dc-4865-9331-a828b12c2bf7/cf99d41f-154f-4525-9df8-a364b4903864"
-					(reference "#PWR051")
+					(reference "#PWR057")
 					(unit 1)
 				)
@@
 		(on_board yes)
 		(dnp no)
-		(property "Reference" "R83"
+		(property "Reference" "R81"
 			(at 69.85 65.278 90)
 			(effects
@@
 			(project "controllerForVehicle"
 				(path "/f177fb06-71dc-4865-9331-a828b12c2bf7/cf99d41f-154f-4525-9df8-a364b4903864"
-					(reference "R83")
+					(reference "R81")
 					(unit 1)
 				)
@@
 		(on_board yes)
 		(dnp no)
-		(property "Reference" "R81"
+		(property "Reference" "R79"
 			(at 69.8482 60.198 90)
 			(effects
@@
 			(project "controllerForVehicle"
 				(path "/f177fb06-71dc-4865-9331-a828b12c2bf7/cf99d41f-154f-4525-9df8-a364b4903864"
-					(reference "R81")
+					(reference "R79")
 					(unit 1)
 				)
@@
 		(on_board yes)
 		(dnp no)
-		(property "Reference" "R73"
+		(property "Reference" "R70"
 			(at 69.85 39.878 90)
 			(effects
@@
 			(project "controllerForVehicle"
 				(path "/f177fb06-71dc-4865-9331-a828b12c2bf7/cf99d41f-154f-4525-9df8-a364b4903864"
-					(reference "R73")
+					(reference "R70")
 					(unit 1)
 				)
@@
 		(on_board yes)
 		(dnp no)
-		(property "Reference" "R80"
+		(property "Reference" "R78"
 			(at 69.85 57.658 90)
 			(effects
@@
 			(project "controllerForVehicle"
 				(path "/f177fb06-71dc-4865-9331-a828b12c2bf7/cf99d41f-154f-4525-9df8-a364b4903864"
-					(reference "R80")
+					(reference "R78")
 					(unit 1)
 				)
@@
 		(on_board yes)
 		(dnp no)
-		(property "Reference" "R78"
+		(property "Reference" "R75"
 			(at 69.85 50.038 90)
 			(effects
@@
 			(project "controllerForVehicle"
 				(path "/f177fb06-71dc-4865-9331-a828b12c2bf7/cf99d41f-154f-4525-9df8-a364b4903864"
-					(reference "R78")
+					(reference "R75")
 					(unit 1)
 				)
@@
 		(on_board yes)
 		(dnp no)
-		(property "Reference" "R76"
+		(property "Reference" "R73"
 			(at 69.85 47.498 90)
 			(effects
@@
 			(project "controllerForVehicle"
 				(path "/f177fb06-71dc-4865-9331-a828b12c2bf7/cf99d41f-154f-4525-9df8-a364b4903864"
-					(reference "R76")
+					(reference "R73")
 					(unit 1)
 				)
@@
 		(on_board yes)
 		(dnp no)
-		(property "Reference" "R77"
+		(property "Reference" "R74"
 			(at 133.35 53.34 90)
 			(effects
@@
 			(project "controllerForVehicle"
 				(path "/f177fb06-71dc-4865-9331-a828b12c2bf7/cf99d41f-154f-4525-9df8-a364b4903864"
-					(reference "R77")
+					(reference "R74")
 					(unit 1)
 				)
@@
 		(on_board yes)
 		(dnp no)
-		(property "Reference" "R84"
+		(property "Reference" "R77"
 			(at 23.114 54.864 0)
 			(effects
@@
 			(project "controllerForVehicle"
 				(path "/f177fb06-71dc-4865-9331-a828b12c2bf7/cf99d41f-154f-4525-9df8-a364b4903864"
-					(reference "R84")
+					(reference "R77")
 					(unit 1)
 				)
@@
 		(dnp no)
 		(fields_autoplaced yes)
-		(property "Reference" "#PWR049"
+		(property "Reference" "#PWR055"
 			(at 59.69 13.97 0)
 			(effects
@@
 			(project "controllerForVehicle"
 				(path "/f177fb06-71dc-4865-9331-a828b12c2bf7/cf99d41f-154f-4525-9df8-a364b4903864"
-					(reference "#PWR049")
+					(reference "#PWR055")
 					(unit 1)
 				)
@@
 		(on_board yes)
 		(dnp no)
-		(property "Reference" "R82"
+		(property "Reference" "R80"
 			(at 69.8482 62.738 90)
 			(effects
@@
 			(project "controllerForVehicle"
 				(path "/f177fb06-71dc-4865-9331-a828b12c2bf7/cf99d41f-154f-4525-9df8-a364b4903864"
-					(reference "R82")
+					(reference "R80")
 					(unit 1)
 				)
@@
 		(on_board yes)
 		(dnp no)
-		(property "Reference" "R68"
+		(property "Reference" "R65"
 			(at 133.35 31.75 90)
 			(effects
@@
 			(project "controllerForVehicle"
 				(path "/f177fb06-71dc-4865-9331-a828b12c2bf7/cf99d41f-154f-4525-9df8-a364b4903864"
-					(reference "R68")
+					(reference "R65")
 					(unit 1)
 				)
@@
 		(on_board yes)
 		(dnp no)
-		(property "Reference" "R69"
+		(property "Reference" "R66"
 			(at 25.654 30.734 0)
 			(effects
@@
 			(project "controllerForVehicle"
 				(path "/f177fb06-71dc-4865-9331-a828b12c2bf7/cf99d41f-154f-4525-9df8-a364b4903864"
-					(reference "R69")
+					(reference "R66")
 					(unit 1)
 				)
@@
 		(dnp no)
 		(fields_autoplaced yes)
-		(property "Reference" "#PWR050"
+		(property "Reference" "#PWR056"
 			(at 142.24 49.53 0)
 			(effects
@@
 			(project "controllerForVehicle"
 				(path "/f177fb06-71dc-4865-9331-a828b12c2bf7/cf99d41f-154f-4525-9df8-a364b4903864"
-					(reference "#PWR050")
+					(reference "#PWR056")
 					(unit 1)
 				)
@@
 		(on_board yes)
 		(dnp no)
-		(property "Reference" "R72"
+		(property "Reference" "R69"
 			(at 133.35 41.91 90)
 			(effects
@@
 			(project "controllerForVehicle"
 				(path "/f177fb06-71dc-4865-9331-a828b12c2bf7/cf99d41f-154f-4525-9df8-a364b4903864"
-					(reference "R72")
+					(reference "R69")
 					(unit 1)
 				)
@@
 		(on_board yes)
 		(dnp no)
-		(property "Reference" "R74"
+		(property "Reference" "R71"
 			(at 69.85 42.418 90)
 			(effects
@@
 			(project "controllerForVehicle"
 				(path "/f177fb06-71dc-4865-9331-a828b12c2bf7/cf99d41f-154f-4525-9df8-a364b4903864"
-					(reference "R74")
+					(reference "R71")
 					(unit 1)
 				)
@@
 		(on_board yes)
 		(dnp no)
-		(property "Reference" "R70"
+		(property "Reference" "R67"
 			(at 69.85 34.798 90)
 			(effects
@@
 			(project "controllerForVehicle"
 				(path "/f177fb06-71dc-4865-9331-a828b12c2bf7/cf99d41f-154f-4525-9df8-a364b4903864"
-					(reference "R70")
+					(reference "R67")
 					(unit 1)
 				)
@@
 		(on_board yes)
 		(dnp no)
-		(property "Reference" "R71"
+		(property "Reference" "R68"
 			(at 69.85 37.338 90)
 			(effects
@@
 			(project "controllerForVehicle"
 				(path "/f177fb06-71dc-4865-9331-a828b12c2bf7/cf99d41f-154f-4525-9df8-a364b4903864"
-					(reference "R71")
-					(unit 1)
-				)
+					(reference "R68")
+					(unit 1)
+				)
