File: mcu_esp32.kicad_sch (KiCad schematic)
At the start: 23 parts, among them SW2 IO0, SW3 EN, T1 S8050, T2 S8050, U5 ESP32-WROOM-32D, U6 CP2102N-Axx-xQFN28

Commit message: silinecek
Parts:
- renumbered C14 to C12, C15 to C13, C16 to C14, C17 to C15, C18 to C16, C19 to C17, C20 to C18, C21 to C19, C22 to C20, R8 to R14, R9 to R15, R11 to R16, R12 to R17, R13 to R18, R14 to R19, R15 to R20, R16 to R21
Changed lines of the file:
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@@
 		(dnp no)
 		(fields_autoplaced yes)
-		(property "Reference" "#PWR021"
+		(property "Reference" "#PWR017"
 			(at 78.74 62.23 0)
 			(effects
@@
 			(project "controllerForVehicle"
 				(path "/f177fb06-71dc-4865-9331-a828b12c2bf7/0ded9e45-71e1-4118-a2b1-0d1586a9cfb7"
-					(reference "#PWR021")
+					(reference "#PWR017")
 					(unit 1)
 				)
@@
 		(dnp no)
 		(fields_autoplaced yes)
-		(property "Reference" "R11"
+		(property "Reference" "R16"
 			(at 93.98 40.64 90)
 			(effects
@@
 			(project "controllerForVehicle"
 				(path "/f177fb06-71dc-4865-9331-a828b12c2bf7/0ded9e45-71e1-4118-a2b1-0d1586a9cfb7"
-					(reference "R11")
+					(reference "R16")
 					(unit 1)
 				)
@@
 		(dnp no)
 		(fields_autoplaced yes)
-		(property "Reference" "#PWR022"
+		(property "Reference" "#PWR018"
 			(at 78.74 88.9 0)
 			(effects
@@
 			(project "controllerForVehicle"
 				(path "/f177fb06-71dc-4865-9331-a828b12c2bf7/0ded9e45-71e1-4118-a2b1-0d1586a9cfb7"
-					(reference "#PWR022")
+					(reference "#PWR018")
 					(unit 1)
 				)
@@
 		(dnp no)
 		(fields_autoplaced yes)
-		(property "Reference" "R9"
+		(property "Reference" "R15"
 			(at 130.81 29.2099 0)
 			(effects
@@
 			(project "controllerForVehicle"
 				(path "/f177fb06-71dc-4865-9331-a828b12c2bf7/0ded9e45-71e1-4118-a2b1-0d1586a9cfb7"
-					(reference "R9")
+					(reference "R15")
 					(unit 1)
 				)
@@
 		(dnp no)
 		(fields_autoplaced yes)
-		(property "Reference" "C17"
+		(property "Reference" "C15"
 			(at 191.77 21.5835 0)
 			(effects
@@
 			(project "controllerForVehicle"
 				(path "/f177fb06-71dc-4865-9331-a828b12c2bf7/0ded9e45-71e1-4118-a2b1-0d1586a9cfb7"
-					(reference "C17")
+					(reference "C15")
 					(unit 1)
 				)
@@
 		(dnp no)
 		(fields_autoplaced yes)
-		(property "Reference" "#PWR020"
+		(property "Reference" "#PWR016"
 			(at 160.02 55.88 0)
 			(effects
@@
 			(project "controllerForVehicle"
 				(path "/f177fb06-71dc-4865-9331-a828b12c2bf7/0ded9e45-71e1-4118-a2b1-0d1586a9cfb7"
-					(reference "#PWR020")
+					(reference "#PWR016")
 					(unit 1)
 				)
@@
 		(dnp no)
 		(fields_autoplaced yes)
-		(property "Reference" "R15"
+		(property "Reference" "R20"
 			(at 175.26 76.2 90)
 			(effects
@@
 			(project "controllerForVehicle"
 				(path "/f177fb06-71dc-4865-9331-a828b12c2bf7/0ded9e45-71e1-4118-a2b1-0d1586a9cfb7"
-					(reference "R15")
+					(reference "R20")
 					(unit 1)
 				)
@@
 		(dnp no)
 		(fields_autoplaced yes)
-		(property "Reference" "R14"
+		(property "Reference" "R19"
 			(at 93.98 67.31 90)
 			(effects
@@
 			(project "controllerForVehicle"
 				(path "/f177fb06-71dc-4865-9331-a828b12c2bf7/0ded9e45-71e1-4118-a2b1-0d1586a9cfb7"
-					(reference "R14")
+					(reference "R19")
 					(unit 1)
 				)
@@
 		(dnp no)
 		(fields_autoplaced yes)
-		(property "Reference" "C16"
+		(property "Reference" "C14"
 			(at 182.88 21.5835 0)
 			(effects
@@
 			(project "controllerForVehicle"
 				(path "/f177fb06-71dc-4865-9331-a828b12c2bf7/0ded9e45-71e1-4118-a2b1-0d1586a9cfb7"
-					(reference "C16")
+					(reference "C14")
 					(unit 1)
 				)
@@
 		(dnp no)
 		(fields_autoplaced yes)
-		(property "Reference" "C22"
+		(property "Reference" "C20"
 			(at 83.8136 74.93 90)
 			(effects
@@
 			(project "controllerForVehicle"
 				(path "/f177fb06-71dc-4865-9331-a828b12c2bf7/0ded9e45-71e1-4118-a2b1-0d1586a9cfb7"
-					(reference "C22")
+					(reference "C20")
 					(unit 1)
 				)
@@
 		(dnp no)
 		(fields_autoplaced yes)
-		(property "Reference" "#PWR024"
+		(property "Reference" "#PWR020"
 			(at 36.83 100.33 0)
 			(effects
@@
 			(project "controllerForVehicle"
 				(path "/f177fb06-71dc-4865-9331-a828b12c2bf7/0ded9e45-71e1-4118-a2b1-0d1586a9cfb7"
-					(reference "#PWR024")
+					(reference "#PWR020")
 					(unit 1)
 				)
@@
 		(dnp no)
 		(fields_autoplaced yes)
-		(property "Reference" "#PWR018"
+		(property "Reference" "#PWR014"
 			(at 83.82 31.75 0)
 			(effects
@@
 			(project "controllerForVehicle"
 				(path "/f177fb06-71dc-4865-9331-a828b12c2bf7/0ded9e45-71e1-4118-a2b1-0d1586a9cfb7"
-					(reference "#PWR018")
+					(reference "#PWR014")
 					(unit 1)
 				)
@@
 		(dnp no)
 		(fields_autoplaced yes)
-		(property "Reference" "C19"
+		(property "Reference" "C17"
 			(at 162.56 45.7135 0)
 			(effects
@@
 			(project "controllerForVehicle"
 				(path "/f177fb06-71dc-4865-9331-a828b12c2bf7/0ded9e45-71e1-4118-a2b1-0d1586a9cfb7"
-					(reference "C19")
+					(reference "C17")
 					(unit 1)
 				)
@@
 		(dnp no)
 		(fields_autoplaced yes)
-		(property "Reference" "C14"
+		(property "Reference" "C12"
 			(at 86.36 21.5835 0)
 			(effects
@@
 			(project "controllerForVehicle"
 				(path "/f177fb06-71dc-4865-9331-a828b12c2bf7/0ded9e45-71e1-4118-a2b1-0d1586a9cfb7"
-					(reference "C14")
+					(reference "C12")
 					(unit 1)
 				)
@@
 		(on_board yes)
 		(dnp no)
-		(property "Reference" "R13"
+		(property "Reference" "R18"
 			(at 123.19 73.914 90)
 			(effects
@@
 			(project "controllerForVehicle"
 				(path "/f177fb06-71dc-4865-9331-a828b12c2bf7/0ded9e45-71e1-4118-a2b1-0d1586a9cfb7"
-					(reference "R13")
+					(reference "R18")
 					(unit 1)
 				)
@@
 		(dnp no)
 		(fields_autoplaced yes)
-		(property "Reference" "C21"
+		(property "Reference" "C19"
 			(at 83.8136 48.26 90)
 			(effects
@@
 			(project "controllerForVehicle"
 				(path "/f177fb06-71dc-4865-9331-a828b12c2bf7/0ded9e45-71e1-4118-a2b1-0d1586a9cfb7"
-					(reference "C21")
+					(reference "C19")
 					(unit 1)
 				)
@@
 		(dnp no)
 		(fields_autoplaced yes)
-		(property "Reference" "#PWR023"
+		(property "Reference" "#PWR019"
 			(at 201.93 97.79 0)
 			(effects
@@
 			(project "controllerForVehicle"
 				(path "/f177fb06-71dc-4865-9331-a828b12c2bf7/0ded9e45-71e1-4118-a2b1-0d1586a9cfb7"
-					(reference "#PWR023")
+					(reference "#PWR019")
 					(unit 1)
 				)
@@
 		(dnp no)
 		(fields_autoplaced yes)
-		(property "Reference" "R12"
+		(property "Reference" "R17"
 			(at 123.19 49.53 90)
 			(effects
@@
 			(project "controllerForVehicle"
 				(path "/f177fb06-71dc-4865-9331-a828b12c2bf7/0ded9e45-71e1-4118-a2b1-0d1586a9cfb7"
-					(reference "R12")
+					(reference "R17")
 					(unit 1)
 				)
@@
 		(dnp no)
 		(fields_autoplaced yes)
-		(property "Reference" "#PWR019"
+		(property "Reference" "#PWR015"
 			(at 128.27 46.99 0)
 			(effects
@@
 			(project "controllerForVehicle"
 				(path "/f177fb06-71dc-4865-9331-a828b12c2bf7/0ded9e45-71e1-4118-a2b1-0d1586a9cfb7"
-					(reference "#PWR019")
+					(reference "#PWR015")
 					(unit 1)
 				)
@@
 		(dnp no)
 		(fields_autoplaced yes)
-		(property "Reference" "C20"
+		(property "Reference" "C18"
 			(at 171.45 45.7135 0)
 			(effects
@@
 			(project "controllerForVehicle"
 				(path "/f177fb06-71dc-4865-9331-a828b12c2bf7/0ded9e45-71e1-4118-a2b1-0d1586a9cfb7"
-					(reference "C20")
+					(reference "C18")
 					(unit 1)
 				)
@@
 		(dnp no)
 		(fields_autoplaced yes)
-		(property "Reference" "R8"
+		(property "Reference" "R14"
 			(at 60.96 22.86 90)
 			(effects
@@
 			(project "controllerForVehicle"
 				(path "/f177fb06-71dc-4865-9331-a828b12c2bf7/0ded9e45-71e1-4118-a2b1-0d1586a9cfb7"
-					(reference "R8")
+					(reference "R14")
 					(unit 1)
 				)
@@
 		(dnp no)
 		(fields_autoplaced yes)
-		(property "Reference" "#PWR017"
+		(property "Reference" "#PWR013"
 			(at 180.34 13.97 0)
 			(effects
@@
 			(project "controllerForVehicle"
 				(path "/f177fb06-71dc-4865-9331-a828b12c2bf7/0ded9e45-71e1-4118-a2b1-0d1586a9cfb7"
-					(reference "#PWR017")
+					(reference "#PWR013")
 					(unit 1)
 				)
@@
 		(dnp no)
 		(fields_autoplaced yes)
-		(property "Reference" "C18"
+		(property "Reference" "C16"
 			(at 130.81 36.8235 0)
 			(effects
@@
 			(project "controllerForVehicle"
 				(path "/f177fb06-71dc-4865-9331-a828b12c2bf7/0ded9e45-71e1-4118-a2b1-0d1586a9cfb7"
-					(reference "C18")
+					(reference "C16")
 					(unit 1)
 				)
@@
 		(dnp no)
 		(fields_autoplaced yes)
-		(property "Reference" "C15"
+		(property "Reference" "C13"
 			(at 95.25 21.5835 0)
 			(effects
@@
 			(project "controllerForVehicle"
 				(path "/f177fb06-71dc-4865-9331-a828b12c2bf7/0ded9e45-71e1-4118-a2b1-0d1586a9cfb7"
-					(reference "C15")
+					(reference "C13")
 					(unit 1)
 				)
@@
 		(on_board yes)
 		(dnp no)
-		(property "Reference" "R16"
+		(property "Reference" "R21"
 			(at 175.26 86.36 90)
 			(effects
@@
 			(project "controllerForVehicle"
 				(path "/f177fb06-71dc-4865-9331-a828b12c2bf7/0ded9e45-71e1-4118-a2b1-0d1586a9cfb7"
-					(reference "R16")
-					(unit 1)
-				)
+					(reference "R21")
+					(unit 1)
+				)
