File: power.kicad_sch (KiCad schematic)
At the start: 39 parts, among them IC1 MP2338GTL-Z, U2 AMS1117-3.3, U3 LM7805_TO220

Commit message: added components
servo controller, esp32
Parts:
- removed U3: LM7805_TO220, Package_TO_SOT_THT:TO-220-3_Vertical, symbol Regulator_Linear:LM7805_TO220
- added U7: L7805, Package_TO_SOT_SMD:TO-252-2, symbol Regulator_Linear:L7805
- IC1: footprint MP2338GTLZ -> MP2338GTL-Z:MP2338GTLZ
- PS1: footprint SOIC127P600X170-9N -> TPS54531DDAR:SOIC127P600X170-9N
- renumbered C5 to C23, C6 to C24, C8 to C25, C3 to C26, C4 to C27, C1 to C28, C2 to C29, C9 to C30, C10 to C31, C7 to C32, C11 to C33, C16 to C34, C19 to C35, C20 to C36, C12 to C37, C13 to C38, C14 to C39, C17 to C40, C18 to C41, C15 to C42, D1 to D25, R1 to R19, R5 to R20, R2 to R21, R3 to R22, R6 to R23, R4 to R24, R10 to R25, R7 to R26, R11 to R27, R8 to R28, R9 to R29, R12 to R30, U2 to U8
Connections:
- net 5V1: now also U7.3 (OUT)
- net GND: now also U7.2 (GND)
- net VIN: now also U7.1 (IN)

Commit message: Visual Improvements
Other:
- moved on the sheet: C23, C24, C25, C28, C29, C30, C31, C32, C33, C34, C35, C36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

Commit message: schematic finished
Parts:
- L1: footprint (none) -> Inductor_SMD:L_Coilcraft_XAL6060-XXX
- renumbered C26 to C23, C27 to C24, C28 to C25, C29 to C26, C23 to C27, C24 to C28, C25 to C29, R19 to R25, R20 to R26, R21 to R27, R22 to R28, R23 to R29, R24 to R30, R25 to R31, R26 to R32, R27 to R33, R28 to R34, R29 to R35, R30 to R36

Commit message: silinecek
Parts:
- renumbered C23 to C21, C24 to C22, C25 to C23, C26 to C24, C27 to C25, C28 to C26, C29 to C27, C30 to C28, C31 to C29, C32 to C30, C33 to C31, C34 to C32, C35 to C33, C36 to C34, C37 to C35, C38 to C36, C39 to C37, C40 to C38, C41 to C39, C42 to C40, R25 to R28, R26 to R29, R27 to R30, R28 to R31, R29 to R32, R30 to R33, R31 to R34, R32 to R35, R33 to R36, R34 to R37, R35 to R38, R36 to R39
