File: servo_control.kicad_sch (KiCad schematic)
At the start: 17 parts, among them U9 PCA9685PW

Commit message: silinecek
Parts:
- removed R51, R54, R56, R57, R61, R65: 10k, Resistor_SMD:R_0805_2012Metric, symbol Device:R_Small
- added RN1, RN2: 10K, Resistor_THT:R_Array_SIP4, symbol Device:R_Network03_Split
- renumbered R52 to R55, R53 to R56, R55 to R58
Connections:
- net GND: now also RN1.2 (R1.2), RN1.3 (R2.2), RN1.4 (R3.2), RN2.2 (R1.2), RN2.3 (R2.2), RN2.4 (R3.2)
- net PCA_A0: now also RN1.1 (R1)
- net PCA_A1: now also RN1.1 (R1)
- net PCA_A2: now also RN1.1 (R1)
- net PCA_A3: now also RN2.1 (R1)
- net PCA_A4: now also RN2.1 (R1)
- net PCA_A5: now also RN2.1 (R1)
