File: com.kicad_sch (KiCad schematic)
At the start: 6 parts

Commit message: esp32 silindi, yerleştirmeler yapıldı
Parts:
- removed R19, R20: 22R, Resistor_SMD:R_0805_2012Metric, symbol Device:R_Small
Other:
- note removed: "STM32 ESP32 Comm"
