File: controllerForVehicle.kicad_pcb (KiCad board)
At the start: 4 copper layers, 203 parts, among them IC1 MP2338GTL-Z, J1 Debug, J10 Conn_01x02, J11 Conn_01x02, J12 Conn_01x02, J13 USB_C_Receptacle_PowerOnly_6P, J14 USB_C_Receptacle_USB2.0_16P, J15 USB_C_Receptacle_USB2.0_16P, J2 Boot_Sel, J3 VIN, J4 Conn_01x08, J5 Conn_01x08, J6 Conn_01x08, J7 Conn_01x02, J8 Conn_01x02, J9 Conn_01x02, SW1 RESET, SW2 IO0, SW3 EN, T1 S8050, T2 S8050, U1 STM32F103C8Tx, U10 MPU6050, U11 MCP23S17_SO, U2 L298N, U3 L298N, U4 L298N, U5 ESP32-WROOM-32D, U6 CP2102N-Axx-xQFN28, U7 L7805, U8 AMS1117-3.3, U9 PCA9685PW, Y1 8mHz

Commit message: esp32 silindi, yerleştirmeler yapıldı
Parts:
- removed C13: 220uF 35V, Capacitor_SMD:CP_Elec_8x10.5
- removed C14: 100u, Capacitor_SMD:C_0805_2012Metric
- removed C15, C17, C20: 0.1u, Capacitor_SMD:C_0805_2012Metric
- removed C16, C19: 10u, Capacitor_SMD:C_0805_2012Metric
- removed C18, C21, C22: 1n / 50V, Capacitor_SMD:C_0805_2012Metric
- removed D26, D31: 1N5819, Diode_SMD:D_SOD-123
- removed D27, D28, D29, D30: ESD05V88D-LC, Diode_SMD:D_SOD-882
- removed D32, D33, D34, D35, D36, D37, D38, D39: 1N4007, Diode_SMD:D_SOD-123
- removed J15: USB_C_Receptacle_USB2.0_16P, Connector_USB:USB_C_Receptacle_Palconn_UTC16-G
- removed R11, R14: 470R, Resistor_SMD:R_0805_2012Metric
- removed R12, R13: 12K, Resistor_SMD:R_0805_2012Metric
- removed R15, R16: 0R, Resistor_SMD:R_0805_2012Metric
- removed R19, R20: 22R, Resistor_SMD:R_0805_2012Metric
- removed R45, R46, R47, R48: 20R, Resistor_SMD:R_0805_2012Metric
- removed R49, R50: 4.7K, Resistor_SMD:R_0805_2012Metric
- removed R8: 5K, Resistor_SMD:R_0805_2012Metric
- removed R9: 12k, Resistor_SMD:R_0805_2012Metric
- removed SW2: IO0, Button_Switch_SMD:SW_SPST_B3U-1000P
- removed SW3: EN, Button_Switch_SMD:SW_SPST_B3U-1000P
- removed T1, T2: S8050, Package_TO_SOT_SMD:TSOT-23
- removed U5: ESP32-WROOM-32D, RF_Module:ESP32-WROOM-32D
- removed U6: CP2102N-Axx-xQFN28, Package_DFN_QFN:QFN-28-1EP_5x5mm_P0.5mm_EP3.1x3.1mm_ThermalVias
- added C8: 220uF 35V, Capacitor_SMD:CP_Elec_8x10.5, F.Cu at (80.2, 46.5)
- added D17: 1N4007, Diode_SMD:D_SOD-123, F.Cu at (105.5, 32.8)
- added D18: 1N4007, Diode_SMD:D_SOD-123, F.Cu at (105.5, 30.1)
- added D19: 1N4007, Diode_SMD:D_SOD-123, F.Cu at (105.5, 35.6)
- added D20: 1N4007, Diode_SMD:D_SOD-123, F.Cu at (105.5, 38.4)
- added D21: 1N4007, Diode_SMD:D_SOD-123, F.Cu at (88.7, 35.6)
- added D22: 1N4007, Diode_SMD:D_SOD-123, F.Cu at (88.6, 38.4)
- added D23: 1N4007, Diode_SMD:D_SOD-123, F.Cu at (88.7, 32.8)
- added D24: 1N4007, Diode_SMD:D_SOD-123, F.Cu at (88.6, 30.1)
- J14: value USB_C_Receptacle_USB2.0_16P -> STM_UART; footprint Connector_USB:USB_C_Receptacle_Palconn_UTC16-G -> Connector_PinHeader_2.54mm:PinHeader_1x04_P2.54mm_Vertical
- moved JP7 301.1 mm to (43.1, 66.4), turned to 0 degrees
- moved R84 299.9 mm to (34.8, 61.0), turned to -90 degrees
- moved JP8 297.8 mm to (43.1, 69.2), turned to 0 degrees
- moved R68 297.0 mm to (47.4, 66.4), turned to 180 degrees
- moved JP9 294.6 mm to (43.1, 72.1), turned to 0 degrees
- moved R72 294.4 mm to (47.3, 69.2), turned to 180 degrees
- moved U11 293.4 mm to (30.4, 69.1), turned to 90 degrees
- moved R77 291.8 mm to (47.3, 72.0), turned to 180 degrees
- moved R24 291.0 mm to (-48.6, 63.8), turned to -90 degrees
- moved R23 287.9 mm to (-45.6, 63.8), turned to -90 degrees
- moved R22 284.9 mm to (-42.7, 63.8), turned to -90 degrees
- moved R53 284.5 mm to (60.9, 82.9), turned to 0 degrees
- moved R55 284.3 mm to (65.0, 83.8), turned to 90 degrees
- moved C46 282.9 mm to (32.3, 77.8)
- moved C47 282.7 mm to (30.1, 77.8)
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Connections:
- D1 pad 2: DC1_1 -> DC3_1
- D10 pad 1: DC1_2 -> DC5_1
- D11 pad 1: DC2_1 -> VIN
- D11 pad 2: GND -> DC5_2
- D12 pad 1: DC2_2 -> DC5_2
- D13 pad 1: DC5_1 -> VIN
- D13 pad 2: GND -> DC6_1
- D14 pad 1: DC5_2 -> DC6_1
- D15 pad 1: DC6_1 -> VIN
- D15 pad 2: GND -> DC6_2
- D2 pad 1: VIN -> DC3_1
- D2 pad 2: DC1_2 -> GND
- D3 pad 2: DC2_1 -> DC3_2
- D4 pad 1: VIN -> DC3_2
- D4 pad 2: DC2_2 -> GND
- D5 pad 2: DC5_1 -> DC4_1
- D6 pad 1: VIN -> DC4_1
- D6 pad 2: DC5_2 -> GND
- D7 pad 2: DC6_1 -> DC4_2
- D8 pad 1: VIN -> DC4_2
- D8 pad 2: DC6_2 -> GND
- D9 pad 1: DC1_1 -> VIN
- D9 pad 2: GND -> DC5_1
- J1 pad 2: SWCLK -> SWDIO
- J1 pad 3: SWDIO -> SWCLK
- J10 pad 1: DC3_2 -> DC3_1
- J10 pad 2: DC3_1 -> DC3_2
- J11 pad 1: DC2_2 -> DC2_1
- J11 pad 2: DC2_1 -> DC2_2
- J12 pad 1: DC1_2 -> DC1_1
- J12 pad 2: DC1_1 -> DC1_2
- J7 pad 1: DC6_2 -> DC6_1
- J7 pad 2: DC6_1 -> DC6_2
- J8 pad 1: DC5_2 -> DC5_1
- J8 pad 2: DC5_1 -> DC5_2
- J9 pad 1: DC4_2 -> DC4_1
- J9 pad 2: DC4_1 -> DC4_2
- R10 pad 2: DCEn1 -> DCEn3
- R17 pad 2: DCEn2 -> DCEn4
- R18 pad 2: DCEn3 -> DCEn5
- R58 pad 2: DCEn4 -> DCEn6
- R59 pad 2: DCEn5 -> DCEn1
- R60 pad 2: DCEn6 -> DCEn2
- U1 pad 32: USB_D- -> unconnected-(U1-PA11-Pad32)
- U1 pad 33: USB_D+ -> unconnected-(U1-PA12-Pad33)
- U2 pad 10: DCIn2_1 -> DCIn4_1
- U2 pad 12: DCIn2_2 -> DCIn4_2
- U2 pad 13: DC2_1 -> DC4_1
- U2 pad 14: DC2_2 -> DC4_2
- U2 pad 2: DC1_1 -> DC3_1
- U2 pad 3: DC1_2 -> DC3_2
- U2 pad 5: DCIn1_1 -> DCIn3_2
- U2 pad 7: DCIn1_2 -> DCIn3_1
- U3 pad 10: DCIn4_1 -> DCIn6_1
- U3 pad 12: DCIn4_2 -> DCIn6_2
- U3 pad 13: DC4_1 -> DC6_1
- U3 pad 14: DC5_2 -> DC6_2
- U3 pad 2: DC3_1 -> DC5_1
- U3 pad 3: DC3_2 -> DC5_2
- U3 pad 5: DCIn3_1 -> DCIn5_1
- U3 pad 7: DCIn3_2 -> DCIn5_2
- U4 pad 10: DCIn6_1 -> DCIn2_1
- U4 pad 12: DCIn6_2 -> DCIn2_2
- U4 pad 13: DC6_1 -> DC2_1
- U4 pad 14: DC6_2 -> DC2_2
- U4 pad 2: DC5_1 -> DC1_1
- U4 pad 3: DC5_2 -> DC1_2
- U4 pad 5: DCIn5_1 -> DCIn1_1
- U4 pad 7: DCIn5_2 -> DCIn1_2
Routing:
- net EN: track 41.2 -> 0.00 mm, vias 2 -> 0
- net IO0: track 29.5 -> 0.00 mm
- net DC2_1: track 18.9 -> 0.00 mm
- net MCP_A2: track 0.00 -> 14.6 mm
- net DC2_2: track 14.6 -> 0.00 mm
- net RESET: track 20.6 -> 6.05 mm
- net DCIn6_1: track 14.1 -> 0.00 mm
- net DCIn6_2: track 14.0 -> 0.00 mm
- net Net-(D26-A): track 13.0 -> 0.00 mm
- net MCP_A1: track 0.00 -> 12.1 mm
- net ESP_D+: track 11.7 -> 0.00 mm
- net Net-(U4-EnA): track 10.4 -> 0.00 mm
- net 5V1: track 10.2 -> 0.00 mm
- net RXD: track 9.36 -> 0.00 mm
- net 3V3: track 28.2 -> 18.9 mm
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Other:
- board outline added: 99.4 x 99.6 mm

Commit message: dc sürücü yol çizimleri yapıldı
Parts:
- moved R21 89.4 mm to (48.5, 78.8)
- moved R22 89.4 mm to (45.5, 78.8)
- moved R24 89.4 mm to (39.6, 78.8)
- moved R23 89.4 mm to (42.5, 78.8)
- moved R79 45.4 mm to (100.0, 37.3), turned to 90 degrees
- moved R70 44.5 mm to (59.1, 53.4), turned to -90 degrees
- moved R78 40.9 mm to (97.5, 37.3), turned to 90 degrees
- moved R71 39.7 mm to (61.7, 53.4), turned to -90 degrees
- moved R73 33.3 mm to (68.0, 37.3), turned to 90 degrees
- moved R74 33.3 mm to (65.5, 37.3), turned to 90 degrees
- moved R75 29.4 mm to (91.2, 53.4), turned to -90 degrees
- moved R76 29.4 mm to (93.7, 53.4), turned to -90 degrees
- moved D6 10.7 mm to (62.4, 30.3), turned to 0 degrees
- moved D14 10.5 mm to (28.9, 30.3), turned to 0 degrees
- moved D20 10.2 mm to (99.2, 30.3), turned to 180 degrees
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Connections:
- R70 pad 1: DCIn1_1 -> DCIn4_2
- R71 pad 1: DCIn1_2 -> DCIn4_1
- R73 pad 1: DCIn2_1 -> DCIn3_2
- R74 pad 1: DCIn2_2 -> DCIn3_1
- R75 pad 1: DCIn3_1 -> DCIn2_2
- R76 pad 1: DCIn3_2 -> DCIn2_1
- R78 pad 1: DCIn4_1 -> DCIn1_2
- R79 pad 1: DCIn4_2 -> DCIn1_1
Routing:
- net VIN: track 0.00 -> 328.3 mm, vias 0 -> 60
- net GND: track 0.00 -> 111.2 mm, vias 0 -> 100
- net DC1_1: track 0.00 -> 102.5 mm
- net DC3_1: track 0.00 -> 102.5 mm
- net Net-(U11-GPB6): track 0.00 -> 96.4 mm, vias 0 -> 2
- net Net-(U11-GPB7): track 0.00 -> 96.2 mm, vias 0 -> 2
- net Net-(U11-GPB5): track 0.00 -> 75.8 mm, vias 0 -> 2
- net Net-(U11-GPB4): track 0.00 -> 74.2 mm, vias 0 -> 2
- net Net-(U11-GPB3): track 0.00 -> 69.1 mm, vias 0 -> 2
- net Net-(U11-GPB2): track 0.00 -> 68.9 mm, vias 0 -> 2
- net DC4_1: track 0.00 -> 63.8 mm
- net DC2_1: track 0.00 -> 63.8 mm
- net DC1_2: track 0.00 -> 61.1 mm
- net DC3_2: track 0.00 -> 61.1 mm
- net Net-(U11-GPB1): track 0.00 -> 48.6 mm, vias 0 -> 2
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- added copper zone on In2.Cu, net 3V3
- added copper zone on F.Cu, net GND
- added copper zone on In1.Cu, net GND
- added copper zone on F.Cu, net VIN
- added copper zone on In2.Cu, net VIN

Commit message: yerleştirmeler devam
Parts:
- moved C23 77.4 mm to (157.1, 89.0)
- moved C25 77.4 mm to (146.3, 94.5)
- moved C26 77.4 mm to (136.3, 94.5)
- moved U7 77.4 mm to (152.0, 93.6)
- moved U8 77.4 mm to (141.3, 91.8)
- moved C24 77.4 mm to (146.9, 89.0)
- moved C44 50.6 mm to (65.0, 153.9)
- moved C45 50.6 mm to (62.6, 153.9)
- moved R67 50.6 mm to (63.8, 147.6)
- moved R66 50.6 mm to (63.8, 150.1)
- moved U10 50.6 mm to (58.2, 137.4)
- moved R65 29.6 mm to (65.1, 72.5)
- moved R51 29.6 mm to (51.4, 72.5)
- moved R54 29.6 mm to (54.1, 72.5)
- moved R56 29.6 mm to (56.9, 72.5)
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Connections:
- U9 pad 17: DCEn6 -> DCEn1
- U9 pad 18: DCEn5 -> DCEn2
- U9 pad 19: DCEn4 -> DCEn3
- U9 pad 20: DCEn3 -> DCEn4
- U9 pad 21: DCEn2 -> DCEn5
- U9 pad 22: DCEn1 -> DCEn6
Routing:
- net DCEn6: track 0.00 -> 52.8 mm, vias 0 -> 2
- net DCEn2: track 0.00 -> 47.7 mm, vias 0 -> 2
- net DCEn1: track 0.00 -> 43.4 mm
- net GND: track 111.2 -> 154.5 mm, vias 100 -> 144
- net PCA_7: track 0.00 -> 42.0 mm, vias 0 -> 2
- net PCA_6: track 0.00 -> 40.7 mm, vias 0 -> 2
- net PCA_5: track 0.00 -> 38.8 mm, vias 0 -> 2
- net PCA_4: track 0.00 -> 34.9 mm, vias 0 -> 2
- net PCA_3: track 0.00 -> 33.9 mm, vias 0 -> 2
- net DCEn5: track 0.00 -> 31.3 mm
- net DCEn4: track 0.00 -> 31.0 mm, vias 0 -> 2
- net PCA_2: track 0.00 -> 31.0 mm, vias 0 -> 2
- net PCA_1: track 0.00 -> 27.5 mm, vias 0 -> 2
- net 5V2: track 0.00 -> 24.5 mm
- net PCA_0: track 0.00 -> 24.2 mm, vias 0 -> 2
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