File: L298N.kicad_sch (KiCad schematic)
At the start: 12 parts, among them U2 L298N

Commit message: Routing
Parts:
- added R49, R50, R6, R7: 100R, Resistor_SMD:R_0805_2012Metric, symbol Device:R_Small
Connections:
- net DCIn1_1: now also R6.2; no longer U2.5 (IN1)
- net DCIn1_2: now also R7.2; no longer U2.7 (IN2)
- net DCIn2_1: now also R49.2; no longer U2.10 (IN3)
- net DCIn2_2: now also R50.2; no longer U2.12 (IN4)
- new net: R6.1, U2.5 (IN1)
- new net: R50.1, U2.12 (IN4)
- new net: R7.1, U2.7 (IN2)
- new net: R49.1, U2.10 (IN3)
